Commit message: V1 Architecture Complete: Flex Sensors, IK Engine, ML Pipeline, and Optical Tracking

File: visualizer/public/robot.urdf (robot description, URDF)
Before this commit: robot mime_arm, 2 links, 1 joints
Links:
- added link index_link; visual box size=0.02 0.02 0.1
- added link thumb_link; visual box size=0.02 0.02 0.1
Joints:
- added joint index_joint: type revolute, parent arm_link, child index_link, origin xyz=-0.06 0 0.3 rpy=0 0 0, axis 0 1 0, limit lower=0 upper=1.57 effort=10 velocity=3
- added joint thumb_joint: type revolute, parent arm_link, child thumb_link, origin xyz=0.06 0 0.3 rpy=0 0 0, axis 0 1 0, limit lower=-1.57 upper=0 effort=10 velocity=3
